File: hw/touchsynth/touch_led.kicad_sch (KiCad schematic)
At the start: 62 parts, among them U5 CD4051B, U6 CD4051B, U7 74HC595, U8 74HC595, U9 74HC595

Commit message: Schematic v2: hand-drawn sheet layouts with wires; MIDI in DNP
- draw.py/gen_sch2.py/layouts.py: placement + wiring per block, automatic
  labels for remaining split nets, short detection, junctions, KiCad
  endpoint-only connection semantics
- all 7 sheets laid out (ladder drawn as a transistor stack, diff amps,
  integrator with reset, R-2R DAC, ...); ERC 0 violations, netlist == design,
  145 simulated elements match
- MIDI input parts marked DNP (footprints kept)
- docs/touchsynth_schematic.pdf

Co-Authored-By: Claude Opus 5.5 (1M context) <noreply@anthropic.com>
Connections:
- net DAC_N0: no longer names the net of R16.1, R17.2, R18.1
- net DAC_N1: no longer names the net of R18.2, R19.2, R20.1
- net DAC_N2: no longer names the net of R20.2, R21.2, R22.1
- net DAC_N3: no longer names the net of R22.2, R23.2, R24.1
- net DAC_N4: no longer names the net of R24.2, R25.2, R26.1
- net DAC_N5: no longer names the net of R26.2, R27.2, R28.1
- net DAC_N6: no longer names the net of R28.2, R29.2, R30.1
Other:
- note added: "LEDs (4.7k arrays, ~0.6 mA each)"
- note added: "Shift registers (daisy-chained: LEDs 0-7, LEDs 8-15, trim DAC)"
- note added: "Touch multiplexers (select S0...S2 shared with the 74HC595 data / clock)"
- note added: "Touch pads (copper under solder mask)"
- note added: "VCA trim DAC: 8-bit R-2R ladder (R = 100k, 2R = 200k), output impedance 100k"
- note removed: "LEDs"
- note removed: "Shift registers (LEDs + trim DAC)"
- note removed: "Touch multiplexers"
- note removed: "Touch pads"
- note removed: "VCA trim DAC (8-bit R-2R)"

Commit message: PCB placement by functional block, silkscreen art, discrete LED resistors
- gen_pcb.py / pcb_place.py: 100 x 100 mm 2-layer board; keys, LEDs, connectors and test points fixed,
  ICs anchored per block, remaining parts placed greedily by connectivity inside their block
- blocks tile the circuit area with a 0.35 mm street for the dashed silkscreen frames and a reserved
  title tab each (pcb_art.py); piano keybed with hatched black keys; logo, resonant saw and ladder
  response curves on the front; signal-flow diagram on the back
- LED resistor arrays replaced by 16 discrete 4.7k 0603 (basic part) next to each LED
- deterministic schematic UUIDs, net name labels for PCB parity, op-amp re-pairing, fab.py

Co-Authored-By: Claude Opus 5.5 (1M context) <noreply@anthropic.com>
Parts:
- removed RN1, RN2, RN3, RN4: 4.7k x4, Resistor_SMD:R_Array_Convex_4x0603, symbol Device:R_Pack04
- added R32, R33, R35, R37, R39, R41, R43, R45, R47: 200k, Resistor_SMD:R_0603_1608Metric, symbol Device:R
- added R34, R36, R38, R40, R42, R44, R46: 100k, Resistor_SMD:R_0603_1608Metric, symbol Device:R
- R16: value 200k -> 4.7k; LCSC C25811 -> C23162; Note R-2R termination -> LED 0 series
- R17: value 200k -> 4.7k; LCSC C25811 -> C23162; Note (none) -> LED 1 series
- R18: value 100k -> 4.7k; LCSC C25803 -> C23162; Note (none) -> LED 2 series
- R19: value 200k -> 4.7k; LCSC C25811 -> C23162; Note (none) -> LED 3 series
- R20: value 100k -> 4.7k; LCSC C25803 -> C23162; Note (none) -> LED 4 series
- R21: value 200k -> 4.7k; LCSC C25811 -> C23162; Note (none) -> LED 5 series
- R22: value 100k -> 4.7k; LCSC C25803 -> C23162; Note (none) -> LED 6 series
- R23: value 200k -> 4.7k; LCSC C25811 -> C23162; Note (none) -> LED 7 series
- R24: value 100k -> 4.7k; LCSC C25803 -> C23162; Note (none) -> LED 8 series
- R25: value 200k -> 4.7k; LCSC C25811 -> C23162; Note (none) -> LED 9 series
- R26: value 100k -> 4.7k; LCSC C25803 -> C23162; Note (none) -> LED 10 series
- R27: value 200k -> 4.7k; LCSC C25811 -> C23162; Note (none) -> LED 11 series
- R28: value 100k -> 4.7k; LCSC C25803 -> C23162; Note (none) -> LED 12 series
- R29: value 200k -> 4.7k; LCSC C25811 -> C23162; Note (none) -> LED 13 series
- R30: value 100k -> 4.7k; LCSC C25803 -> C23162; Note (none) -> LED 14 series
- R31: value 200k -> 4.7k; LCSC C25811 -> C23162; Note (none) -> LED 15 series
Connections:
- net DAC_Q0: now also R33.1; no longer R17.1
- net DAC_Q1: now also R35.1; no longer R19.1
- net DAC_Q2: now also R37.1; no longer R21.1
- net DAC_Q3: now also R39.1; no longer R23.1
- net DAC_Q4: now also R41.1; no longer R25.1
- net DAC_Q5: now also R43.1; no longer R27.1
- net DAC_Q6: now also R45.1; no longer R29.1
- net DAC_Q7: now also R47.1; no longer R31.1
- net GND: now also R32.2; no longer R16.2
- net LED_A0: now also R16.2
- net LED_A1: now also R17.2
- net LED_A10: now also R26.2
- net LED_A11: now also R27.2
- net LED_A12: now also R28.2
- net LED_A13: now also R29.2
- net LED_A14: now also R30.2
- net LED_A15: now also R31.2
- net LED_A2: now also R18.2
- net LED_A3: now also R19.2
- net LED_A4: now also R20.2
- net LED_A5: now also R21.2
- net LED_A6: now also R22.2
- net LED_A7: now also R23.2
- net LED_A8: now also R24.2
- net LED_A9: now also R25.2
- net LED_Q0: now also R16.1
- net LED_Q1: now also R17.1
- net LED_Q10: now also R26.1
- net LED_Q11: now also R27.1
- net LED_Q12: now also R28.1
- net LED_Q13: now also R29.1
- net LED_Q14: now also R30.1
- net LED_Q15: now also R31.1
- net LED_Q2: now also R18.1
- net LED_Q3: now also R19.1
- net LED_Q4: now also R20.1
- net LED_Q5: now also R21.1
- net LED_Q6: now also R22.1
- net LED_Q7: now also R23.1
- net LED_Q8: now also R24.1
- net LED_Q9: now also R25.1
- net VTRIM: now also R46.2, R47.2; no longer R30.2, R31.2
- new net DAC_N0: R32.1, R33.2, R34.1
- new net DAC_N1: R34.2, R35.2, R36.1
- new net DAC_N2: R36.2, R37.2, R38.1
- new net DAC_N3: R38.2, R39.2, R40.1
- new net DAC_N4: R40.2, R41.2, R42.1
- new net DAC_N5: R42.2, R43.2, R44.1
- new net DAC_N6: R44.2, R45.2, R46.1
Other:
- note added: "LEDs (4.7k series resistors, ~0.6 mA each)"
- note removed: "LEDs (4.7k arrays, ~0.6 mA each)"
